File: elec/stepper_controllers/_autosave-stepper_controllers.sch (KiCad schematic (older format))
At the start: 28 parts

Commit message: undersoek
Parts:
- added U?: Teensy4.1-teensy, symbol stepper_controllers-rescue:Teensy4.1-teensy
Changed lines of the file:
@@
 	1    0    0    -1
 $EndComp
+$Comp
+L stepper_controllers-rescue:Teensy4.1-teensy U?
+U 1 1 62C008D8
+P 5850 3100
+F 0 "U?" V 5804 5528 50  0000 L CNN
+F 1 "Teensy4.1-teensy" V 5895 5528 50  0000 L CNN
+F 2 "" H 5450 3500 50  0001 C CNN
+F 3 "" H 5450 3500 50  0001 C CNN
+	1    5850 3100
+	0    1    1    0
+$EndComp
 $EndSCHEMATC
