File: elec/stepper_controllers/stepper_controllers.sch (KiCad schematic (older format))
At the start: 28 parts

Commit message: kicad
Parts:
- added J? (x8): Conn_01x04_Male, symbol Connector:Conn_01x04_Male
- added U?: Teensy4.1-teensy, symbol stepper_controllers-rescue:Teensy4.1-teensy
- added U? (x4): 74HC595, symbol 74xx:74HC595
- A?: value Pololu_Breakout_A4988 -> stepper 00
- A?: value Pololu_Breakout_A4988 -> stepper 01
- A?: value Pololu_Breakout_A4988 -> stepper 02
- A?: value Pololu_Breakout_A4988 -> stepper 03
- A?: value Pololu_Breakout_A4988 -> stepper 04
- A?: value Pololu_Breakout_A4988 -> stepper 05
- A?: value Pololu_Breakout_A4988 -> stepper 08
- A?: value Pololu_Breakout_A4988 -> stepper 09
- A?: value Pololu_Breakout_A4988 -> stepper 10
- A?: value Pololu_Breakout_A4988 -> stepepr 11
- A?: value Pololu_Breakout_A4988 -> stepepr 12
- A?: value Pololu_Breakout_A4988 -> stepper 13
- A?: value Pololu_Breakout_A4988 -> stepper 06
- A?: value Pololu_Breakout_A4988 -> stepper 07
- A?: value Pololu_Breakout_A4988 -> stepper 14
- A?: value Pololu_Breakout_A4988 -> stepper 15
- J?: value Conn_01x16_Male -> SWITCHES CONNECTOR
Connections:
- wire segments 207 -> 456
Other:
- moved on the sheet: A?, J?, R?
